File: schematic/iron.sch (EAGLE design)
At the start: 62 parts, among them IC1 LD117AS18TR, IC2 MCP602SN, IC3 STM32F103C8T, Q1 TCP8107, SW1 EC12E_SW

Commit message: final
Connections:
- removed net N$23: R24.1, SW1G$2.2
- new net PB5: IC3MCU.PB5, R24.1, SW1G$2.2
Changed lines of the file:
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@@
 <?xml version="1.0" encoding="utf-8"?>
 <!DOCTYPE eagle SYSTEM "eagle.dtd">
-<eagle version="8.2.1">
+<eagle version="8.3.2">
 <drawing>
 <settings>
 <setting alwaysvectorfont="no"/>
+<setting keepoldvectorfont="yes"/>
 <setting verticaltext="up"/>
 </settings>
@@
 </segment>
 </net>
-<net name="N$23" class="0">
-<segment>
-<pinref part="R24" gate="G$1" pin="1"/>
-<pinref part="SW1" gate="G$2" pin="2"/>
-<wire x1="195.58" y1="-50.8" x2="200.66" y2="-50.8" width="0.1524" layer="91"/>
-<wire x1="200.66" y1="-50.8" x2="200.66" y2="-45.72" width="0.1524" layer="91"/>
-</segment>
-</net>
 <net name="PB0" class="0">
 <segment>
@@
 </segment>
 </net>
+<net name="PB5" class="0">
+<segment>
+<pinref part="IC3" gate="MCU" pin="PB5"/>
+<wire x1="208.28" y1="33.02" x2="223.52" y2="33.02" width="0.1524" layer="91"/>
+<label x="213.36" y="33.02" size="1.778" layer="95"/>
+</segment>
+<segment>
+<pinref part="R24" gate="G$1" pin="1"/>
+<pinref part="SW1" gate="G$2" pin="2"/>
+<wire x1="195.58" y1="-50.8" x2="200.66" y2="-50.8" width="0.1524" layer="91"/>
+<wire x1="200.66" y1="-50.8" x2="200.66" y2="-45.72" width="0.1524" layer="91"/>
+<wire x1="195.58" y1="-50.8" x2="195.58" y2="-58.42" width="0.1524" layer="91"/>
+<wire x1="195.58" y1="-58.42" x2="203.2" y2="-58.42" width="0.1524" layer="91"/>
+<label x="200.66" y="-58.42" size="1.778" layer="95"/>
+</segment>
+</net>
 </nets>
 </sheet>
@@
 <compatibility>
 <note version="8.2" severity="warning">
-Since Version 8.2, Eagle supports online libraries. The ids
+Since Version 8.2, EAGLE supports online libraries. The ids
 of those online libraries will not be understood (or retained)
 with this version.
